File: expansionboard.brd (EAGLE design)
At the start: 160 x 110 mm, 40 parts, among them IC2 REG1117, IC3 REG1117, U1 LAN951X, X1 J1012F21R, Y1 20Mhz

Commit message: for now, a complete logic board and expansion board until I find something wrong with it
Parts:
- added C12, C13: (no value), SparkFun-Capacitors:CAP-PTH-SMALLEZ
- added C14, C15, C19, C20: 0.1uf, SparkFun-Capacitors:1206
- added C18: 4.7uf, SparkFun-Capacitors:1206
- added JP1: USB-A-S, SparkFun-Connectors:USB-A-S
- added R8: (no value), SparkFun-Resistors:1206
- added R9: 0ohm, SparkFun-Resistors:1206
- added X2, X3, X4: PCI-60-POS-145167, con-amp:145167-2
- moved R7 185.5 mm to (134.3, 47.0), turned to 315 degrees
- moved C9 170.1 mm to (126.4, 27.6), turned to 270 degrees
- moved C8 167.4 mm to (129.2, 27.6), turned to 270 degrees
- moved C7 164.6 mm to (132.1, 27.6), turned to 270 degrees
- moved C6 161.9 mm to (134.9, 27.6), turned to 270 degrees
- moved R4 155.2 mm to (131.8, 39.1), turned to 45 degrees
- moved R3 154.9 mm to (133.3, 37.5), turned to 45 degrees
- moved R2 154.7 mm to (134.9, 35.9), turned to 45 degrees
- moved R1 154.6 mm to (136.5, 34.0), turned to 45 degrees
- moved R5 51.4 mm to (153.4, 13.2), turned to 0 degrees
- moved C11 28.7 mm to (127.6, 49.5), turned to 315 degrees
- moved C10 28.5 mm to (123.7, 45.6), turned to 315 degrees
- moved Y1 21.4 mm to (129.2, 41.9), turned to 225 degrees
- moved R6 5.83 mm to (123.8, 27.9)
- moved U1 1.59 mm to (117.8, 39.1)
Connections:
- removed net 3.3V_AN: R1.P$2, R2.P$2, R3.P$2, R4.P$2
- new net N$27: U1.45
- new net USB2+: U1.2, X2.1, X2.2
- new net USB2-: U1.1, X2.3, X2.4
- new net USB2_PWR: U1.14, X2.5, X2.6
- new net USB3+: U1.4, X3.1, X3.2
- new net USB3-: U1.3, X3.3, X3.4
- new net USB3_PWR: U1.16, X3.5, X3.6
- new net USB4+: U1.7, X4.1, X4.2
- new net USB4-: U1.6, X4.3, X4.4
- new net USB4_PWR: U1.17, X4.5, X4.6
- new net USB5+: JP1.D+, U1.9
- new net USB5-: JP1.D-, U1.8
- new net USB5_PWR: JP1.VBUS, U1.18
- new net VBUS_DET: R8.1, U1.11
- new net VDD18CORE: C18.1, C19.1, C20.1, U1.15, U1.38
- new net VDDA33: C14.1, C15.1, R1.P$2, R2.P$2, R3.P$2, R4.P$2, R9.2
- net 3.3V: now also C12.1, C13.1, R8.2, R9.1, U1.10, U1.19, U1.27, U1.33, U1.39, U1.46, U1.49, U1.5, U1.51, U1.54, U1.57, U1.64
- net 5V: now also X2.13, X2.14, X2.15, X2.16, X2.17, X2.18, X3.13, X3.14, X3.15, X3.16, X3.17, X3.18, X4.13, X4.14, X4.15, X4.16, X4.17, X4.18
- net GND: now also C12.2, C13.2, C14.2, C15.2, C18.2, C19.2, C20.2, JP1.GND, X2.10, X2.11, X2.115, X2.116, X2.117, X2.118, X2.119, X2.12, X2.120, X2.7, X2.8, X2.9, X3.10, X3.11, X3.115, X3.116, X3.117, X3.118, X3.119, X3.12, X3.120, X3.7, X3.8, X3.9, X4.10, X4.11, X4.115, X4.116, X4.117, X4.118, X4.119, X4.12, X4.120, X4.7, X4.8, X4.9
- net GPIO10: now also X2.45, X2.46, X3.45, X3.46, X4.45, X4.46
- net GPIO11: now also X2.47, X2.48, X3.47, X3.48, X4.47, X4.48
- net GPIO12: now also X2.49, X2.50, X3.49, X3.50, X4.49, X4.50
- net GPIO13: now also X2.51, X2.52, X3.51, X3.52, X4.51, X4.52
- net GPIO17: now also X2.57, X2.58, X3.57, X3.58, X4.57, X4.58
- net GPIO18: now also X2.59, X2.60, X3.59, X3.60, X4.59, X4.60
- net GPIO19: now also X2.61, X2.62, X3.61, X3.62, X4.61, X4.62
- net GPIO20: now also X2.63, X2.64, X3.63, X3.64, X4.63, X4.64
- net GPIO21: now also X2.65, X2.66, X3.65, X3.66, X4.65, X4.66
- net GPIO22: now also X2.67, X2.68, X3.67, X3.68, X4.67, X4.68
- net GPIO23: now also X2.69, X2.70, X3.69, X3.70, X4.69, X4.70
- net GPIO24: now also X2.71, X2.72, X3.71, X3.72, X4.71, X4.72
- net GPIO25: now also X2.73, X2.74, X3.73, X3.74, X4.73, X4.74
- net GPIO26: now also X2.75, X2.76, X3.75, X3.76, X4.75, X4.76
- net GPIO27: now also X2.77, X2.78, X3.77, X3.78, X4.77, X4.78
- net GPIO28: now also X2.79, X2.80, X3.79, X3.80, X4.79, X4.80
- net GPIO29: now also X2.81, X2.82, X3.81, X3.82, X4.81, X4.82
- net GPIO30: now also X2.83, X2.84, X3.83, X3.84, X4.83, X4.84
- net GPIO31: now also X2.85, X2.86, X3.85, X3.86, X4.85, X4.86
- net GPIO32: now also X2.87, X2.88, X3.87, X3.88, X4.87, X4.88
- net GPIO33: now also X2.89, X2.90, X3.89, X3.90, X4.89, X4.90
- net GPIO34: now also X2.91, X2.92, X3.91, X3.92, X4.91, X4.92
- net GPIO35: now also X2.93, X2.94, X3.93, X3.94, X4.93, X4.94
- net GPIO36: now also X2.95, X2.96, X3.95, X3.96, X4.95, X4.96
- net GPIO37: now also X2.97, X2.98, X3.97, X3.98, X4.97, X4.98
- net GPIO38: now also X2.100, X2.99, X3.100, X3.99, X4.100, X4.99
- net GPIO39: now also X2.101, X2.102, X3.101, X3.102, X4.101, X4.102
- net GPIO4: now also X2.33, X2.34, X3.33, X3.34, X4.33, X4.34
- net GPIO40: now also X2.103, X2.104, X3.103, X3.104, X4.103, X4.104
- net GPIO41: now also X2.105, X2.106, X3.105, X3.106, X4.105, X4.106
- net GPIO42: now also X2.107, X2.108, X3.107, X3.108, X4.107, X4.108
- net GPIO43: now also X2.109, X2.110, X3.109, X3.110, X4.109, X4.110
- net GPIO44: now also X2.111, X2.112, X3.111, X3.112, X4.111, X4.112
- net GPIO45: now also X2.113, X2.114, X3.113, X3.114, X4.113, X4.114
- net GPIO5: now also X2.35, X2.36, X3.35, X3.36, X4.35, X4.36
- net GPIO6: now also X2.37, X2.38, X3.37, X3.38, X4.37, X4.38
- net GPIO7: now also X2.39, X2.40, X3.39, X3.40, X4.39, X4.40
- net GPIO8: now also X2.41, X2.42, X3.41, X3.42, X4.41, X4.42
- net GPIO9: now also X2.43, X2.44, X3.43, X3.44, X4.43, X4.44
- net RXD0: now also X2.55, X2.56, X3.55, X3.56, X4.55, X4.56
- net SCL: now also X2.27, X2.28, X3.27, X3.28, X4.27, X4.28
- net SCL1: now also X2.31, X2.32, X3.31, X3.32, X4.31, X4.32
- net SDA: now also X2.25, X2.26, X3.25, X3.26, X4.25, X4.26
- net SDA1: now also X2.29, X2.30, X3.29, X3.30, X4.29, X4.30
- net TXD0: now also X2.53, X2.54, X3.53, X3.54, X4.53, X4.54
- net USB+: now also U1.59
- net USB-: now also U1.58
- net V+: now also X2.19, X2.20, X2.21, X2.22, X2.23, X2.24, X3.19, X3.20, X3.21, X3.22, X3.23, X3.24, X4.19, X4.20, X4.21, X4.22, X4.23, X4.24
Routing:
- net V+: track 22.2 -> 422.9 mm
- net 3.3V: track 6.21 -> 340.5 mm, vias 0 -> 1
- net 5V: track 57.9 -> 386.7 mm
- net USB+: track 0.00 -> 179.8 mm, vias 0 -> 1
- net USB-: track 0.00 -> 179.5 mm, vias 0 -> 1
- net SCL1: track 0.00 -> 122.1 mm
- net SCL: track 0.00 -> 120.5 mm
- net GPIO5: track 0.00 -> 119.4 mm
- net GPIO7: track 0.00 -> 118.9 mm
- net GPIO9: track 0.00 -> 118.0 mm
- net SDA1: track 0.00 -> 113.3 mm
- net SDA: track 0.00 -> 112.1 mm
- net GPIO6: track 0.00 -> 112.0 mm
- net GPIO4: track 0.00 -> 111.9 mm
- net GPIO8: track 0.00 -> 110.1 mm
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Other:
- outline, holes or cut-outs redrawn
